Commit message: sync https://www.lejuhub.com/highlydynamic/kuavo-ros-control/commit/bb386b93a3527457c267722d238989565b72e616

File: src/kuavo_assets/models/biped_s40/urdf/biped_s40.urdf (robot description, URDF)
Before this commit: robot biped_s4, 45 links, 44 joints
Links:
- link head: geometry collision mesh filename=package://kuavo_assets/models/biped_s40/meshes/head_pitch.S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; visual mesh filename=package://kuavo_assets/models/biped_s40/meshes/head_pitch.S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
- link neck_motor: geometry collision mesh filename=package://kuavo_assets/models/biped_s40/meshes/head_yaw.STL; visual mesh filename=package://kuavo_assets/models/biped_s40/meshes/head_yaw.STL

File: src/kuavo_assets/models/biped_s41/urdf/biped_s41.urdf (robot description, URDF)
Before this commit: robot biped_s41, 45 links, 44 joints
Links:
- link head: geometry collision mesh filename=package://kuavo_assets/models/biped_s41/meshes/head_pitch.S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; visual mesh filename=package://kuavo_assets/models/biped_s41/meshes/head_pitch.S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
- link neck_motor: geometry collision mesh filename=package://kuavo_assets/models/biped_s41/meshes/head_yaw.STL; visual mesh filename=package://kuavo_assets/models/biped_s41/meshes/head_yaw.STL

File: src/kuavo_assets/models/biped_s42/urdf/biped_s42.urdf (robot description, URDF)
Before this commit: robot biped_s42, 45 links, 44 joints
Links:
- added link radar, mass 0.26880; collision mesh filename=package://kuavo_assets/models/biped_s42/meshes/radar.STL; visual mesh filename=package://kuavo_assets/models/biped_s42/meshes/radar.STL
- link base_link: mass 25.1666 -> 24.6469
- link camera: mass 0.0170256015508834 -> 0.04700
- link head: mass 0.604629406788488 -> 0.54920; geometry collision mesh filename=package://kuavo_assets/models/biped_s42/meshes/head_pitch.S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; visual mesh filename=package://kuavo_assets/models/biped_s42/meshes/head_pitch.S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
- link neck_motor: mass 0.0736988170113863 -> 0.35000000; geometry collision mesh filename=package://kuavo_assets/models/biped_s42/meshes/head_yaw.STL; visual mesh filename=package://kuavo_assets/models/biped_s42/meshes/head_yaw.STL
Joints:
- added joint radar: type fixed, parent head, child radar, origin xyz=0.0217799337881943 0 0.105417258037133 rpy=0 0.229686043245049 0
- joint camera: axis 0.565415371333248 -0.245538929357162 0.787411005784073 -> (none)

File: src/kuavo_assets/models/biped_s43/urdf/biped_s43.urdf (robot description, URDF)
Before this commit: robot biped_s4, 45 links, 44 joints
Links:
- link head: geometry collision mesh filename=package://kuavo_assets/models/biped_s43/meshes/head_pitch.S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; visual mesh filename=package://kuavo_assets/models/biped_s43/meshes/head_pitch.S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
- link neck_motor: geometry collision mesh filename=package://kuavo_assets/models/biped_s43/meshes/head_yaw.STL; visual mesh filename=package://kuavo_assets/models/biped_s43/meshes/head_yaw.STL
