Commit message: sync https://www.lejuhub.com/highlydynamic/kuavo-ros-control/commit/1683cb87fe557c72a9fcdbc69d68e002fa78f451

File: src/kuavo_assets/models/biped_s31/urdf/drake/biped_v3.urdf (robot description, URDF)
Before this commit: robot biped_v3, 13 links, 12 joints
Links:
- link torso: geometry visual mesh filename=../../meshes/base_link.STL

File: src/kuavo_assets/models/biped_s31/urdf/drake/biped_v3_full.urdf (robot description, URDF)
Before this commit: robot biped_v3_full, 27 links, 26 joints
Links:
- link torso: geometry visual mesh filename=../../meshes/base_link.STL

File: src/kuavo_assets/models/biped_s32/urdf/drake/biped_v3_arm.urdf (robot description, URDF)
Before this commit: robot biped_v3_arm, 15 links, 14 joints
Links:
- link torso: geometry visual mesh filename=../../meshes/torso.STL

File: src/kuavo_assets/models/biped_s41/urdf/drake/biped_v3.urdf (robot description, URDF)
Before this commit: robot biped_v3, 13 links, 12 joints
Links:
- link torso: geometry visual mesh filename=../../meshes/base_link.STL

File: src/kuavo_assets/models/biped_s41/urdf/drake/biped_v3_full.urdf (robot description, URDF)
Before this commit: robot biped_v3_full, 27 links, 26 joints
Links:
- link torso: geometry visual mesh filename=../../meshes/base_link.STL

File: src/kuavo_assets/models/biped_s43/urdf/drake/biped_v3.urdf (robot description, URDF)
Before this commit: robot biped_v3, 13 links, 12 joints
Links:
- link torso: geometry visual mesh filename=../../meshes/base_link.STL

File: src/kuavo_assets/models/biped_s43/urdf/drake/biped_v3_all_joint.urdf (robot description, URDF)
Before this commit: robot biped_v3_all_joint, 35 links, 30 joints
Links:
- link torso: geometry visual mesh filename=../../meshes/base_link.STL

File: src/kuavo_assets/models/biped_s43/urdf/drake/biped_v3_arm.urdf (robot description, URDF)
Before this commit: robot biped_v3_arm, 15 links, 14 joints
Links:
- link torso: geometry visual mesh filename=../../meshes/base_link.STL

File: src/kuavo_assets/models/biped_s43/urdf/drake/biped_v3_full.urdf (robot description, URDF)
Before this commit: robot biped_v3_full, 27 links, 26 joints
Links:
- link torso: geometry visual mesh filename=../../meshes/base_link.STL
