Commit message: sync https://www.lejuhub.com/highlydynamic/kuavo-ros-control/commit/522cb99c4870e4d3ae42b80bb19d9daf6145f369

File: src/kuavo_assets/models/biped_s42/urdf/biped_s42.urdf (robot description, URDF)
Before this commit: robot biped_s42, 45 links, 44 joints
Joints:
- joint neck_joint_pitch: axis 0 -1 0 -> 0 1 0

Commit message: sync https://www.lejuhub.com/highlydynamic/kuavo-ros-control/commit/de36cb1a0bc5dac2b457861e0c823493089571e2

File: src/kuavo_assets/models/biped_s42/urdf/biped_s42.urdf (robot description, URDF)
Before this commit: robot biped_s42, 46 links, 45 joints
Links:
- added link camera_base, mass 0.0170256015508834; collision mesh filename=package://kuavo_assets/models/biped_s42/meshes/camera_base.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; visual mesh filename=package://kuavo_assets/models/biped_s42/meshes/camera_base.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
- link base_link: mass 22.92233803 -> 26.32533803
Joints:
- added joint camera_base: type fixed, parent zhead_2_link, child camera_base, origin xyz=0.0828919080642966 0 0.119165137551254 rpy=0 0.488692190558416 0
- joint dummy_to_base_link: type floating -> fixed
