Commit message: sync https://www.lejuhub.com/highlydynamic/kuavo-ros-control/commit/b1aa08f0375f306f93f6978236149035de2cb254

File: src/kuavo_assets/models/biped_s31/urdf/biped_s31.urdf (robot description, URDF)
Before this commit: robot biped_s31, 28 links, 27 joints
Joints:
- joint dummy_to_base_link: type fixed -> floating

File: src/kuavo_assets/models/biped_s32/urdf/biped_s32.urdf (robot description, URDF)
Before this commit: robot biped_s32, 28 links, 27 joints
Joints:
- joint dummy_to_base_link: type fixed -> floating

File: src/kuavo_assets/models/biped_s40/urdf/biped_s40.urdf (robot description, URDF)
Before this commit: robot biped_s40, 46 links, 45 joints
Links:
- removed link camera_base
- link base_link: mass 22.6719 -> 22.6889
Joints:
- removed joint camera_base
- joint dummy_to_base_link: type fixed -> floating

File: src/kuavo_assets/models/biped_s41/urdf/biped_s41.urdf (robot description, URDF)
Before this commit: robot biped_s41, 46 links, 45 joints
Links:
- removed link camera_base
Joints:
- removed joint camera_base
- joint dummy_to_base_link: type fixed -> floating

File: src/kuavo_assets/models/biped_s42/urdf/biped_s42.urdf (robot description, URDF)
Before this commit: robot biped_s42, 47 links, 46 joints
Links:
- removed link camera_base
- link base_link: mass 26.32533803 -> 22.92233803
Joints:
- removed joint camera_base
- joint dummy_to_base_link: type fixed -> floating

File: src/kuavo_assets/models/biped_s42/urdf/drake/biped_v3.urdf (robot description, URDF)
Before this commit: robot biped_v3, 13 links, 12 joints
Links:
- link torso: mass 37.01433803 -> 33.61133803

File: src/kuavo_assets/models/biped_s42/urdf/drake/biped_v3_all_joint.urdf (robot description, URDF)
Before this commit: robot biped_v3_all_joint, 35 links, 30 joints
Links:
- link torso: mass 26.89754316 -> 23.49454316

File: src/kuavo_assets/models/biped_s42/urdf/drake/biped_v3_full.urdf (robot description, URDF)
Before this commit: robot biped_v3_full, 27 links, 26 joints
Links:
- link torso: mass 27.54033803 -> 24.13733803

File: src/kuavo_assets/models/biped_s43/urdf/biped_s43.urdf (robot description, URDF)
Before this commit: robot biped_s43, 46 links, 45 joints
Links:
- removed link camera_base
Joints:
- removed joint camera_base
- joint dummy_to_base_link: type fixed -> floating

File: src/kuavo_assets/models/biped_s43/urdf/drake/biped_v3_all_joint.urdf (robot description, URDF)
Before this commit: robot biped_v3_all_joint, 35 links, 30 joints
Links:
- link zarm_l1_link: geometry visual mesh filename=package://biped_s43/meshes/l_arm_pitch.STL
- link zarm_l2_link: geometry visual mesh filename=package://biped_s43/meshes/l_arm_roll.STL
- link zarm_l3_link: geometry visual mesh filename=package://biped_s43/meshes/l_arm_yaw.STL
- link zarm_l4_link: geometry visual mesh filename=package://biped_s43/meshes/l_forearm.STL
- link zarm_l5_link: geometry visual mesh filename=package://biped_s43/meshes/l_hand_yaw.STL
- link zarm_l6_link: geometry visual mesh filename=package://biped_s43/meshes/l_hand_roll.STL
- link zarm_l7_link: geometry visual mesh filename=package://biped_s43/meshes/l_hand_pitch.STL
- link zarm_r1_link: geometry visual mesh filename=package://biped_s43/meshes/r_arm_pitch.STL
- link zarm_r2_link: geometry visual mesh filename=package://biped_s43/meshes/r_arm_roll.STL
- link zarm_r3_link: geometry visual mesh filename=package://biped_s43/meshes/r_arm_yaw.STL
- link zarm_r4_link: geometry visual mesh filename=package://biped_s43/meshes/r_forearm.STL
- link zarm_r5_link: geometry visual mesh filename=package://biped_s43/meshes/r_hand_yaw.STL
- link zarm_r6_link: geometry visual mesh filename=package://biped_s43/meshes/r_hand_roll.STL
- link zarm_r7_link: geometry visual mesh filename=package://biped_s43/meshes/r_hand_pitch.STL

File: src/kuavo_assets/models/biped_s43/urdf/drake/biped_v3_arm.urdf (robot description, URDF)
Before this commit: robot biped_v3_arm, 15 links, 14 joints
Links:
- link zarm_l1_link: geometry visual mesh filename=package://biped_s43/meshes/l_arm_pitch.STL
- link zarm_l2_link: geometry visual mesh filename=package://biped_s43/meshes/l_arm_roll.STL
- link zarm_l3_link: geometry visual mesh filename=package://biped_s43/meshes/l_arm_yaw.STL
- link zarm_l4_link: geometry visual mesh filename=package://biped_s43/meshes/l_forearm.STL
- link zarm_l5_link: geometry visual mesh filename=package://biped_s43/meshes/l_hand_yaw.STL
- link zarm_l6_link: geometry visual mesh filename=package://biped_s43/meshes/l_hand_roll.STL
- link zarm_l7_link: geometry visual mesh filename=package://biped_s43/meshes/l_hand_pitch.STL
- link zarm_r1_link: geometry visual mesh filename=package://biped_s43/meshes/r_arm_pitch.STL
- link zarm_r2_link: geometry visual mesh filename=package://biped_s43/meshes/r_arm_roll.STL
- link zarm_r3_link: geometry visual mesh filename=package://biped_s43/meshes/r_arm_yaw.STL
- link zarm_r4_link: geometry visual mesh filename=package://biped_s43/meshes/r_forearm.STL
- link zarm_r5_link: geometry visual mesh filename=package://biped_s43/meshes/r_hand_yaw.STL
- link zarm_r6_link: geometry visual mesh filename=package://biped_s43/meshes/r_hand_roll.STL
- link zarm_r7_link: geometry visual mesh filename=package://biped_s43/meshes/r_hand_pitch.STL

File: src/kuavo_assets/models/biped_s43/urdf/drake/biped_v3_full.urdf (robot description, URDF)
Before this commit: robot biped_v3_full, 27 links, 26 joints
Links:
- link zarm_l1_link: geometry visual mesh filename=package://biped_s43/meshes/l_arm_pitch.STL
- link zarm_l2_link: geometry visual mesh filename=package://biped_s43/meshes/l_arm_roll.STL
- link zarm_l3_link: geometry visual mesh filename=package://biped_s43/meshes/l_arm_yaw.STL
- link zarm_l4_link: geometry visual mesh filename=package://biped_s43/meshes/l_forearm.STL
- link zarm_l5_link: geometry visual mesh filename=package://biped_s43/meshes/l_hand_yaw.STL
- link zarm_l6_link: geometry visual mesh filename=package://biped_s43/meshes/l_hand_roll.STL
- link zarm_l7_link: geometry visual mesh filename=package://biped_s43/meshes/l_hand_pitch.STL
- link zarm_r1_link: geometry visual mesh filename=package://biped_s43/meshes/r_arm_pitch.STL
- link zarm_r2_link: geometry visual mesh filename=package://biped_s43/meshes/r_arm_roll.STL
- link zarm_r3_link: geometry visual mesh filename=package://biped_s43/meshes/r_arm_yaw.STL
- link zarm_r4_link: geometry visual mesh filename=package://biped_s43/meshes/r_forearm.STL
- link zarm_r5_link: geometry visual mesh filename=package://biped_s43/meshes/r_hand_yaw.STL
- link zarm_r6_link: geometry visual mesh filename=package://biped_s43/meshes/r_hand_roll.STL
- link zarm_r7_link: geometry visual mesh filename=package://biped_s43/meshes/r_hand_pitch.STL

Commit message: sync https://www.lejuhub.com/highlydynamic/kuavo-ros-control/commit/ff25da57ae5d20f50539951ef5ef4efcde454abf

File: src/kuavo_assets/models/biped_s31/urdf/biped_s31.urdf (robot description, URDF)
Before this commit: robot biped_s31, 28 links, 27 joints
Joints:
- joint dummy_to_base_link: type floating -> fixed

File: src/kuavo_assets/models/biped_s32/urdf/biped_s32.urdf (robot description, URDF)
Before this commit: robot biped_s32, 28 links, 27 joints
Joints:
- joint dummy_to_base_link: type floating -> fixed

File: src/kuavo_assets/models/biped_s40/urdf/biped_s40.urdf (robot description, URDF)
Before this commit: robot biped_s40, 45 links, 44 joints
Links:
- added link camera_base, mass 0.0170255961584929; collision mesh filename=package://kuavo_assets/models/biped_s40/meshes/camera_base.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; visual mesh filename=package://kuavo_assets/models/biped_s40/meshes/camera_base.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
- link base_link: mass 22.6889 -> 22.6719
Joints:
- added joint camera_base: type fixed, parent zhead_2_link, child camera_base, origin xyz=0.0766792844154498 0 0.0571889355165869 rpy=0 0.610865238198013 0
- joint dummy_to_base_link: type floating -> fixed

File: src/kuavo_assets/models/biped_s41/urdf/biped_s41.urdf (robot description, URDF)
Before this commit: robot biped_s41, 45 links, 44 joints
Links:
- added link camera_base, mass 0.0170255961584929; collision mesh filename=package://kuavo_assets/models/biped_s41/meshes/camera_base.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; visual mesh filename=package://kuavo_assets/models/biped_s41/meshes/camera_base.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
Joints:
- added joint camera_base: type fixed, parent zhead_2_link, child camera_base, origin xyz=0.0766792844154498 0 0.0571889355165869 rpy=0 0.610865238198013 0
- joint dummy_to_base_link: type floating -> fixed

File: src/kuavo_assets/models/biped_s42/urdf/biped_s42.urdf (robot description, URDF)
Before this commit: robot biped_s42, 46 links, 45 joints
Links:
- added link camera_base, mass 0.0170256015508834; collision mesh filename=package://kuavo_assets/models/biped_s42/meshes/camera_base.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; visual mesh filename=package://kuavo_assets/models/biped_s42/meshes/camera_base.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
- link base_link: mass 22.92233803 -> 26.30833803
Joints:
- added joint camera_base: type fixed, parent zhead_2_link, child camera_base, origin xyz=0.0828919080642966 0 0.119165137551254 rpy=0 0.488692190558416 0
- joint dummy_to_base_link: type floating -> fixed

File: src/kuavo_assets/models/biped_s42/urdf/drake/biped_v3.urdf (robot description, URDF)
Before this commit: robot biped_v3, 13 links, 12 joints
Links:
- link torso: mass 33.61133803 -> 37.01433803

File: src/kuavo_assets/models/biped_s42/urdf/drake/biped_v3_all_joint.urdf (robot description, URDF)
Before this commit: robot biped_v3_all_joint, 35 links, 30 joints
Links:
- link torso: mass 23.49454316 -> 26.89754316

File: src/kuavo_assets/models/biped_s42/urdf/drake/biped_v3_full.urdf (robot description, URDF)
Before this commit: robot biped_v3_full, 27 links, 26 joints
Links:
- link torso: mass 24.13733803 -> 27.54033803

File: src/kuavo_assets/models/biped_s43/urdf/biped_s43.urdf (robot description, URDF)
Before this commit: robot biped_s43, 45 links, 44 joints
Links:
- added link camera_base, mass 0.0170255961584929; collision mesh filename=package://kuavo_assets/models/biped_s43/meshes/camera_base.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; visual mesh filename=package://kuavo_assets/models/biped_s43/meshes/camera_base.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
Joints:
- added joint camera_base: type fixed, parent zhead_2_link, child camera_base, origin xyz=0.0766792844154498 0 0.0571889355165869 rpy=0 0.610865238198013 0
- joint dummy_to_base_link: type floating -> fixed

File: src/kuavo_assets/models/biped_s43/urdf/drake/biped_v3_all_joint.urdf (robot description, URDF)
Before this commit: robot biped_v3_all_joint, 35 links, 30 joints
Links:
- link zarm_l1_link: geometry visual mesh filename=../../meshes/l_arm_pitch.STL
- link zarm_l2_link: geometry visual mesh filename=../../meshes/l_arm_roll.STL
- link zarm_l3_link: geometry visual mesh filename=../../meshes/l_arm_yaw.STL
- link zarm_l4_link: geometry visual mesh filename=../../meshes/l_forearm.STL
- link zarm_l5_link: geometry visual mesh filename=../../meshes/l_hand_yaw.STL
- link zarm_l6_link: geometry visual mesh filename=../../meshes/l_hand_roll.STL
- link zarm_l7_link: geometry visual mesh filename=../../meshes/l_hand_pitch.STL
- link zarm_r1_link: geometry visual mesh filename=../../meshes/r_arm_pitch.STL
- link zarm_r2_link: geometry visual mesh filename=../../meshes/r_arm_roll.STL
- link zarm_r3_link: geometry visual mesh filename=../../meshes/r_arm_yaw.STL
- link zarm_r4_link: geometry visual mesh filename=../../meshes/r_forearm.STL
- link zarm_r5_link: geometry visual mesh filename=../../meshes/r_hand_yaw.STL
- link zarm_r6_link: geometry visual mesh filename=../../meshes/r_hand_roll.STL
- link zarm_r7_link: geometry visual mesh filename=../../meshes/r_hand_pitch.STL

File: src/kuavo_assets/models/biped_s43/urdf/drake/biped_v3_arm.urdf (robot description, URDF)
Before this commit: robot biped_v3_arm, 15 links, 14 joints
Links:
- link zarm_l1_link: geometry visual mesh filename=../../meshes/l_arm_pitch.STL
- link zarm_l2_link: geometry visual mesh filename=../../meshes/l_arm_roll.STL
- link zarm_l3_link: geometry visual mesh filename=../../meshes/l_arm_yaw.STL
- link zarm_l4_link: geometry visual mesh filename=../../meshes/l_forearm.STL
- link zarm_l5_link: geometry visual mesh filename=../../meshes/l_hand_yaw.STL
- link zarm_l6_link: geometry visual mesh filename=../../meshes/l_hand_roll.STL
- link zarm_l7_link: geometry visual mesh filename=../../meshes/l_hand_pitch.STL
- link zarm_r1_link: geometry visual mesh filename=../../meshes/r_arm_pitch.STL
- link zarm_r2_link: geometry visual mesh filename=../../meshes/r_arm_roll.STL
- link zarm_r3_link: geometry visual mesh filename=../../meshes/r_arm_yaw.STL
- link zarm_r4_link: geometry visual mesh filename=../../meshes/r_forearm.STL
- link zarm_r5_link: geometry visual mesh filename=../../meshes/r_hand_yaw.STL
- link zarm_r6_link: geometry visual mesh filename=../../meshes/r_hand_roll.STL
- link zarm_r7_link: geometry visual mesh filename=../../meshes/r_hand_pitch.STL

File: src/kuavo_assets/models/biped_s43/urdf/drake/biped_v3_full.urdf (robot description, URDF)
Before this commit: robot biped_v3_full, 27 links, 26 joints
Links:
- link zarm_l1_link: geometry visual mesh filename=../../meshes/l_arm_pitch.STL
- link zarm_l2_link: geometry visual mesh filename=../../meshes/l_arm_roll.STL
- link zarm_l3_link: geometry visual mesh filename=../../meshes/l_arm_yaw.STL
- link zarm_l4_link: geometry visual mesh filename=../../meshes/l_forearm.STL
- link zarm_l5_link: geometry visual mesh filename=../../meshes/l_hand_yaw.STL
- link zarm_l6_link: geometry visual mesh filename=../../meshes/l_hand_roll.STL
- link zarm_l7_link: geometry visual mesh filename=../../meshes/l_hand_pitch.STL
- link zarm_r1_link: geometry visual mesh filename=../../meshes/r_arm_pitch.STL
- link zarm_r2_link: geometry visual mesh filename=../../meshes/r_arm_roll.STL
- link zarm_r3_link: geometry visual mesh filename=../../meshes/r_arm_yaw.STL
- link zarm_r4_link: geometry visual mesh filename=../../meshes/r_forearm.STL
- link zarm_r5_link: geometry visual mesh filename=../../meshes/r_hand_yaw.STL
- link zarm_r6_link: geometry visual mesh filename=../../meshes/r_hand_roll.STL
- link zarm_r7_link: geometry visual mesh filename=../../meshes/r_hand_pitch.STL
