Commit message: sync https://www.lejuhub.com/highlydynamic/kuavo-ros-control/commit/813672e004c44b5e24f763c9e3156e1d278f97c5

File: src/kuavo_assets/models/biped_s46/urdf/drake/biped_v3.urdf (robot description, URDF)
Before this commit: robot biped_v3, 13 links, 12 joints
Links:
- link torso: mass 38.38963803 -> 38.40663803

File: src/kuavo_assets/models/biped_s46/urdf/drake/biped_v3_all_joint.urdf (robot description, URDF)
Before this commit: robot biped_v3_all_joint, 35 links, 30 joints
Links:
- link torso: mass 27.36284316 -> 27.37984316

File: src/kuavo_assets/models/biped_s46/urdf/drake/biped_v3_full.urdf (robot description, URDF)
Before this commit: robot biped_v3_full, 27 links, 26 joints
Links:
- link torso: mass 28.00563803 -> 28.02263803

File: src/kuavo_assets/models/biped_s48/urdf/drake/biped_v3.urdf (robot description, URDF)
Before this commit: robot biped_v3, 13 links, 12 joints
Links:
- link torso: mass 33.72893803 -> 33.65333803

File: src/kuavo_assets/models/biped_s48/urdf/drake/biped_v3_all_joint.urdf (robot description, URDF)
Before this commit: robot biped_v3_all_joint, 35 links, 30 joints
Links:
- link torso: mass 22.70214316 -> 23.79804316

File: src/kuavo_assets/models/biped_s48/urdf/drake/biped_v3_full.urdf (robot description, URDF)
Before this commit: robot biped_v3_full, 27 links, 26 joints
Links:
- link torso: mass 23.34493803 -> 24.44093803
