Commit message: sync https://www.lejuhub.com/highlydynamic/kuavo-ros-control/commit/36c43be472c1175059c9c009ab92246e1bc5d456

File: src/kuavo_assets/models/biped_s49/urdf/biped_s49.urdf (robot description, URDF)
Before this commit: robot biped_s49, 47 links, 46 joints
Links:
- link base_link: mass 24.42123803 -> 28.34823803
- link camera_base: mass 3.92699081698732E-05 -> 0.0000392699081698732
