Commit message: sync https://www.lejuhub.com/highlydynamic/kuavo-ros-control/commit/e06d1296479e4b2fbe88c4161224f745af661bbc

File: src/kuavo_assets/models/biped_s45/urdf/biped_s45.urdf (robot description, URDF)
Before this commit: robot biped_s45, 53 links, 52 joints
Joints:
- removed joint l_hand_camera
- removed joint l_hand_tripod
- removed joint r_hand_camera
- removed joint r_hand_tripod
- added joint l_hand_camera_joint: type fixed, parent l_hand_tripod, child l_hand_camera, origin xyz=0.11540559159102 -0.0145586110669961 -0.110123491595499 rpy=-1.919862177193763 0.753528063917894 -2.897246568680842, axis 0 0 0
- added joint l_hand_tripod_joint: type fixed, parent zarm_l7_link, child l_hand_tripod, origin xyz=0.0 0.0 0.0 rpy=0.0 0.0 0.0, axis 0 0 0
- added joint r_hand_camera_joint: type fixed, parent r_hand_tripod, child r_hand_camera, origin xyz=0.115405591590931 0.0154312352120435 -0.107724128430896 rpy=1.208853693239594  0.751879414295006 2.888346587751982, axis 0 0 0
- added joint r_hand_tripod_joint: type fixed, parent zarm_r7_link, child r_hand_tripod, origin xyz=0.0 0.0 0.0 rpy=0.0 0.0 0.0, axis 0 0 0

File: src/kuavo_assets/models/biped_s49/urdf/biped_s49.urdf (robot description, URDF)
Before this commit: robot biped_s49, 51 links, 50 joints
Joints:
- removed joint l_hand_camera
- removed joint l_hand_tripod
- removed joint r_hand_camera
- removed joint r_hand_tripod
- added joint l_hand_camera_joint: type fixed, parent l_hand_tripod, child l_hand_camera, origin xyz=0.11540559159102 -0.0145586110669961 -0.110123491595499 rpy=-1.919862177193763 0.753528063917894 -2.897246568680842, axis 0 0 0
- added joint l_hand_tripod_joint: type fixed, parent zarm_l7_link, child l_hand_tripod, origin xyz=0.0 0.0 0.0 rpy=0.0 0.0 0.0, axis 0 0 0
- added joint r_hand_camera_joint: type fixed, parent r_hand_tripod, child r_hand_camera, origin xyz=0.115405591590931 0.0154312352120435 -0.107724128430896 rpy=1.208853693239594  0.751879414295006 2.888346587751982, axis 0 0 0
- added joint r_hand_tripod_joint: type fixed, parent zarm_r7_link, child r_hand_tripod, origin xyz=0.0 0.0 0.0 rpy=0.0 0.0 0.0, axis 0 0 0

Commit message: sync https://www.lejuhub.com/highlydynamic/kuavo-ros-control/commit/f09b657e46500dd8d735e501ac7934e972b5b83a

File: src/kuavo_assets/models/biped_s45/urdf/biped_s45.urdf (robot description, URDF)
Before this commit: robot biped_s45, 53 links, 52 joints
Links:
- link base_link: mass 21.63013803 -> 27.41553803
Joints:
- joint l_hand_camera_joint: origin xyz=0.11540559159102 -0.0145586110669961 -0.110123491595499 rpy=-1.919862177193763 0.753528063917894 -2.897246568680842 -> xyz=0.11540559159102 -0.0145586110669961 -0.110123491595499 rpy=1.919862177193763 0.753528063917894 -2.897246568680842

File: src/kuavo_assets/models/biped_s45/urdf/biped_s45_gazebo.urdf (robot description, URDF)
Before this commit: robot biped_s45, 47 links, 46 joints
Links:
- link base_link: mass 22.11293803 -> 27.89833803

File: src/kuavo_assets/models/biped_s48/urdf/biped_s48.urdf (robot description, URDF)
Before this commit: robot biped_s48, 69 links, 68 joints
Links:
- link base_link: mass 22.11293803 -> 27.41553803

File: src/kuavo_assets/models/biped_s49/urdf/biped_s49.urdf (robot description, URDF)
Before this commit: robot biped_s49, 51 links, 50 joints
Links:
- added link l_Index_prox, mass 0.008; collision mesh filename=package://kuavo_assets/models/biped_s49/meshes/l_Index_prox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; visual mesh filename=package://kuavo_assets/models/biped_s49/meshes/l_Index_prox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
- added link l_index_dist, mass 0.011; collision mesh filename=package://kuavo_assets/models/biped_s49/meshes/l_index_dist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; visual mesh filename=package://kuavo_assets/models/biped_s49/meshes/l_index_dist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
- added link l_little_dist, mass 0.008; collision mesh filename=package://kuavo_assets/models/biped_s49/meshes/l_little_dis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; visual mesh filename=package://kuavo_assets/models/biped_s49/meshes/l_little_dis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
- added link l_little_prox, mass 0.008; collision mesh filename=package://kuavo_assets/models/biped_s49/meshes/l_little_pro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; visual mesh filename=package://kuavo_assets/models/biped_s49/meshes/l_little_pro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
- added link l_middle_dist, mass 0.011; collision mesh filename=package://kuavo_assets/models/biped_s49/meshes/l_middle_dis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; visual mesh filename=package://kuavo_assets/models/biped_s49/meshes/l_middle_dis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
- added link l_middle_prox, mass 0.011; collision mesh filename=package://kuavo_assets/models/biped_s49/meshes/l_middle_pro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; visual mesh filename=package://kuavo_assets/models/biped_s49/meshes/l_middle_pro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
- added link l_palm, mass 0.427; collision mesh filename=package://kuavo_assets/models/biped_s49/meshes/l_palm.STL; visual mesh filename=package://kuavo_assets/models/biped_s49/meshes/l_palm.STL
- added link l_ring_dist, mass 0.008; collision mesh filename=package://kuavo_assets/models/biped_s49/meshes/l_ring_dist.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; visual mesh filename=package://kuavo_assets/models/biped_s49/meshes/l_ring_dist.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
- added link l_ring_prox, mass 0.011; collision mesh filename=package://kuavo_assets/models/biped_s49/meshes/l_ring_prox.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; visual mesh filename=package://kuavo_assets/models/biped_s49/meshes/l_ring_prox.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
- added link l_thumb_dist, mass 0.04; collision mesh filename=package://kuavo_assets/models/biped_s49/meshes/l_thumb_dist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; visual mesh filename=package://kuavo_assets/models/biped_s49/meshes/l_thumb_dist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
- added link l_thumb_prox, mass 0.005; collision mesh filename=package://kuavo_assets/models/biped_s49/meshes/l_thumb_prox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; visual mesh filename=package://kuavo_assets/models/biped_s49/meshes/l_thumb_prox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
- added link r_index_dist, mass 0.011; collision mesh filename=package://kuavo_assets/models/biped_s49/meshes/r_index_dist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; visual mesh filename=package://kuavo_assets/models/biped_s49/meshes/r_index_dist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
- added link r_index_prox, mass 0.008; collision mesh filename=package://kuavo_assets/models/biped_s49/meshes/r_index_prox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; visual mesh filename=package://kuavo_assets/models/biped_s49/meshes/r_index_prox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
- added link r_little_dist, mass 0.008; collision mesh filename=package://kuavo_assets/models/biped_s49/meshes/r_little_dis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; visual mesh filename=package://kuavo_assets/models/biped_s49/meshes/r_little_dis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
- added link r_little_prox, mass 0.008; collision mesh filename=package://kuavo_assets/models/biped_s49/meshes/r_little_pro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; visual mesh filename=package://kuavo_assets/models/biped_s49/meshes/r_little_pro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
- added link r_middle_dist, mass 0.011; collision mesh filename=package://kuavo_assets/models/biped_s49/meshes/r_middle_dis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; visual mesh filename=package://kuavo_assets/models/biped_s49/meshes/r_middle_dis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
- added link r_middle_prox, mass 0.011; collision mesh filename=package://kuavo_assets/models/biped_s49/meshes/r_middle_pro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; visual mesh filename=package://kuavo_assets/models/biped_s49/meshes/r_middle_pro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
- added link r_palm, mass 0.427; collision mesh filename=package://kuavo_assets/models/biped_s49/meshes/r_palm.STL; visual mesh filename=package://kuavo_assets/models/biped_s49/meshes/r_palm.STL
- added link r_ring_dist, mass 0.008; collision mesh filename=package://kuavo_assets/models/biped_s49/meshes/r_ring_dist.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; visual mesh filename=package://kuavo_assets/models/biped_s49/meshes/r_ring_dist.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
- added link r_ring_prox, mass 0.011; collision mesh filename=package://kuavo_assets/models/biped_s49/meshes/r_ring_prox.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; visual mesh filename=package://kuavo_assets/models/biped_s49/meshes/r_ring_prox.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
- added link r_thumb_dist, mass 0.04; collision mesh filename=package://kuavo_assets/models/biped_s49/meshes/r_thumb_dist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; visual mesh filename=package://kuavo_assets/models/biped_s49/meshes/r_thumb_dist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
- added link r_thumb_prox, mass 0.005; collision mesh filename=package://kuavo_assets/models/biped_s49/meshes/r_thumb_prox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; visual mesh filename=package://kuavo_assets/models/biped_s49/meshes/r_thumb_prox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
- link base_link: mass 28.34823803 -> 27.41553803
- link zarm_l7_link: mass 0.64 -> 0.0542110173081966
- link zarm_r7_link: mass 0.64 -> 0.0542110173081966
Joints:
- added joint l_indexMCP: type revolute, parent l_palm, child l_Index_prox, origin xyz=-0.029003 0.088291 0.0022155 rpy=-0.029415 0.05236 0.034907, axis 1 0 0, limit lower=0 upper=1.309 effort=0 velocity=0
- added joint l_indexPIP: type revolute, parent l_Index_prox, child l_index_dist, origin xyz=0 0.035 0 rpy=0.19353 0 0, axis 1 0 0, limit lower=0 upper=1.25 effort=0 velocity=0
- added joint l_littleMCP: type revolute, parent l_palm, child l_little_prox, origin xyz=0.033731 0.083777 0.0022155 rpy=-0.024909 -0.05236 -0.069813, axis 1 0 0, limit lower=0 upper=1.309 effort=0 velocity=0
- added joint l_littlePIP: type revolute, parent l_little_prox, child l_little_dist, origin xyz=0 0.035 0 rpy=0.20294 0 0, axis 1 0 0, limit lower=0 upper=1.25 effort=0 velocity=0
- added joint l_middleMCP: type revolute, parent l_palm, child l_middle_prox, origin xyz=-0.008 0.092284 -0.0017707 rpy=0 0 0, axis 1 0 0, limit lower=0 upper=1.309 effort=0 velocity=0
- added joint l_middlePIP: type revolute, parent l_middle_prox, child l_middle_dist, origin xyz=0 0.042 0 rpy=0.18357 0 0, axis 1 0 0, limit lower=0 upper=1.25 effort=0 velocity=0
- added joint l_palm_fixed_joint: type fixed, parent zarm_l7_link, child l_palm, origin xyz=0 0 -0.07 rpy=-1.57 0 -3.14
- added joint l_ringMCP: type revolute, parent l_palm, child l_ring_prox, origin xyz=0.013103 0.090291 -0.0017845 rpy=-0.0092374 -0.05236 -0.034907, axis 1 0 0, limit lower=0 upper=1.309 effort=0 velocity=0
- added joint l_ringPIP: type revolute, parent l_ring_prox, child l_ring_dist, origin xyz=0 0.042 0 rpy=0.16583 0 0, axis 1 0 0, limit lower=0 upper=1.25 effort=0 velocity=0
- added joint l_thumbCMC: type revolute, parent l_palm, child l_thumb_prox, origin xyz=-0.0245 0.022632 0.023263 rpy=0.14578 -1.0699 -0.12808, axis 0 1 0, limit lower=0 upper=1.5708 effort=0 velocity=0
- added joint l_thumbMCP: type revolute, parent l_thumb_prox, child l_thumb_dist, origin xyz=0 0 0.013647 rpy=0.87266 -0.49642 0, axis -1 0 0, limit lower=0 upper=0.8727 effort=0 velocity=0
- added joint r_indexMCP: type revolute, parent r_palm, child r_index_prox, origin xyz=0.029003 0.088231 -0.0039488 rpy=-0.09929 -0.054667 -0.031168, axis 1 0 0, limit lower=0 upper=1.309 effort=0 velocity=0
- added joint r_indexPIP: type revolute, parent r_index_prox, child r_index_dist, origin xyz=0 0.035 0 rpy=0.19353 0 0, axis 1 0 0, limit lower=0 upper=1.25 effort=0 velocity=0
- added joint r_littleMCP: type revolute, parent r_palm, child r_little_prox, origin xyz=-0.033731 0.083727 -0.0036339 rpy=-0.094666 0.057099 0.065996, axis 1 0 0, limit lower=0 upper=1.309 effort=0 velocity=0
- added joint r_littlePIP: type revolute, parent r_little_prox, child r_little_dist, origin xyz=0 0.035 0 rpy=0.20294 0 0, axis 1 0 0, limit lower=0 upper=1.25 effort=0 velocity=0
- added joint r_middleMCP: type revolute, parent r_palm, child r_middle_prox, origin xyz=0.008 0.091935 -0.0082038 rpy=-0.069813 0 0, axis 1 0 0, limit lower=0 upper=1.309 effort=0 velocity=0
- added joint r_middlePIP: type revolute, parent r_middle_prox, child r_middle_dist, origin xyz=0 0.042 0 rpy=0.18357 0 0, axis 1 0 0, limit lower=0 upper=1.25 effort=0 velocity=0
- added joint r_palm_fixed_joint: type fixed, parent zarm_r7_link, child r_palm, origin xyz=0 0 -0.07 rpy=-1.57 0 0
- added joint r_ringMCP: type revolute, parent r_palm, child r_ring_prox, origin xyz=-0.013103 0.089947 -0.0080786 rpy=-0.079113 0.054667 0.031168, axis 1 0 0, limit lower=0 upper=1.309 effort=0 velocity=0
- added joint r_ringPIP: type revolute, parent r_ring_prox, child r_ring_dist, origin xyz=0 0.042 0 rpy=0.16583 0 0, axis 1 0 0, limit lower=0 upper=1.25 effort=0 velocity=0
- added joint r_thumbCMC: type revolute, parent r_palm, child r_thumb_prox, origin xyz=0.0245 0.0242 0.021628 rpy=0 -0.49642 0, axis 0 -1 0, limit lower=0 upper=1.5708 effort=0 velocity=0
- added joint r_thumbMCP: type revolute, parent r_thumb_prox, child r_thumb_dist, origin xyz=0.013647 0 0 rpy=-0.39332 0.31115 -0.93514, axis 0 0 1, limit lower=0 upper=0.87266 effort=0 velocity=0
- joint l_hand_camera_joint: origin xyz=0.11540559159102 -0.0145586110669961 -0.110123491595499 rpy=-1.919862177193763 0.753528063917894 -2.897246568680842 -> xyz=0.11540559159102 -0.0145586110669961 -0.110123491595499 rpy=1.919862177193763 0.753528063917894 -2.897246568680842

Commit message: sync https://www.lejuhub.com/highlydynamic/kuavo-ros-control/commit/5a297fc5ba9732c435e8605e729a2dee755a432e

File: src/kuavo_assets/models/biped_s45/urdf/biped_s45.urdf (robot description, URDF)
Before this commit: robot biped_s45, 53 links, 52 joints
Links:
- link base_link: mass 27.41553803 -> 21.63013803
Joints:
- joint l_hand_camera_joint: origin xyz=0.11540559159102 -0.0145586110669961 -0.110123491595499 rpy=1.919862177193763 0.753528063917894 -2.897246568680842 -> xyz=0.11540559159102 -0.0145586110669961 -0.110123491595499 rpy=-1.919862177193763 0.753528063917894 -2.897246568680842

File: src/kuavo_assets/models/biped_s45/urdf/biped_s45_gazebo.urdf (robot description, URDF)
Before this commit: robot biped_s45, 47 links, 46 joints
Links:
- link base_link: mass 27.89833803 -> 22.11293803

File: src/kuavo_assets/models/biped_s48/urdf/biped_s48.urdf (robot description, URDF)
Before this commit: robot biped_s48, 69 links, 68 joints
Links:
- link base_link: mass 27.41553803 -> 22.11293803

File: src/kuavo_assets/models/biped_s49/urdf/biped_s49.urdf (robot description, URDF)
Before this commit: robot biped_s49, 73 links, 72 joints
Links:
- removed link l_Index_prox
- removed link l_index_dist
- removed link l_little_dist
- removed link l_little_prox
- removed link l_middle_dist
- removed link l_middle_prox
- removed link l_palm
- removed link l_ring_dist
- removed link l_ring_prox
- removed link l_thumb_dist
- removed link l_thumb_prox
- removed link r_index_dist
- removed link r_index_prox
- removed link r_little_dist
- removed link r_little_prox
- removed link r_middle_dist
- removed link r_middle_prox
- removed link r_palm
- removed link r_ring_dist
- removed link r_ring_prox
- removed link r_thumb_dist
- removed link r_thumb_prox
- link base_link: mass 27.41553803 -> 28.34823803
- link zarm_l7_link: mass 0.0542110173081966 -> 0.64
- link zarm_r7_link: mass 0.0542110173081966 -> 0.64
Joints:
- removed joint l_indexMCP
- removed joint l_indexPIP
- removed joint l_littleMCP
- removed joint l_littlePIP
- removed joint l_middleMCP
- removed joint l_middlePIP
- removed joint l_palm_fixed_joint
- removed joint l_ringMCP
- removed joint l_ringPIP
- removed joint l_thumbCMC
- removed joint l_thumbMCP
- removed joint r_indexMCP
- removed joint r_indexPIP
- removed joint r_littleMCP
- removed joint r_littlePIP
- removed joint r_middleMCP
- removed joint r_middlePIP
- removed joint r_palm_fixed_joint
- removed joint r_ringMCP
- removed joint r_ringPIP
- removed joint r_thumbCMC
- removed joint r_thumbMCP
- joint l_hand_camera_joint: origin xyz=0.11540559159102 -0.0145586110669961 -0.110123491595499 rpy=1.919862177193763 0.753528063917894 -2.897246568680842 -> xyz=0.11540559159102 -0.0145586110669961 -0.110123491595499 rpy=-1.919862177193763 0.753528063917894 -2.897246568680842

File: src/kuavo_assets/models/biped_s49/urdf/biped_s49_gazebo.urdf (robot description, URDF)
Before this commit: robot biped_s49, 69 links, 68 joints
Links:
- removed link l_Index_prox
- removed link l_index_dist
- removed link l_little_dist
- removed link l_little_prox
- removed link l_middle_dist
- removed link l_middle_prox
- removed link l_palm
- removed link l_ring_dist
- removed link l_ring_prox
- removed link l_thumb_dist
- removed link l_thumb_prox
- removed link r_index_dist
- removed link r_index_prox
- removed link r_little_dist
- removed link r_little_prox
- removed link r_middle_dist
- removed link r_middle_prox
- removed link r_palm
- removed link r_ring_dist
- removed link r_ring_prox
- removed link r_thumb_dist
- removed link r_thumb_prox
Joints:
- removed joint l_indexMCP
- removed joint l_indexPIP
- removed joint l_littleMCP
- removed joint l_littlePIP
- removed joint l_middleMCP
- removed joint l_middlePIP
- removed joint l_palm_fixed_joint
- removed joint l_ringMCP
- removed joint l_ringPIP
- removed joint l_thumbCMC
- removed joint l_thumbMCP
- removed joint r_indexMCP
- removed joint r_indexPIP
- removed joint r_littleMCP
- removed joint r_littlePIP
- removed joint r_middleMCP
- removed joint r_middlePIP
- removed joint r_palm_fixed_joint
- removed joint r_ringMCP
- removed joint r_ringPIP
- removed joint r_thumbCMC
- removed joint r_thumbMCP
