Commit message: sync https://www.lejuhub.com/highlydynamic/kuavo-ros-control/commit/2160e2c9b7c81e692dca73e156d39ae30f47270c

File: src/kuavo_assets/models/biped_s53/urdf/biped_s53_gazebo.urdf (robot description, URDF)
Before this commit: robot biped_s53, 48 links, 47 joints
Links:
- link waist_yaw_link: mass 21.63516 -> 20.63616

File: src/kuavo_assets/models/biped_s53/urdf/drake/biped_v3.urdf (robot description, URDF)
Before this commit: robot biped_v3, 14 links, 13 joints
Links:
- link waist_yaw_link: mass 34.54246 -> 33.54346

File: src/kuavo_assets/models/biped_s53/urdf/drake/biped_v3_all_joint.urdf (robot description, URDF)
Before this commit: robot biped_v3_all_joint, 35 links, 30 joints
Links:
- link torso: mass 39.42094316 -> 38.42194316

File: src/kuavo_assets/models/biped_s53/urdf/drake/biped_v3_full.urdf (robot description, URDF)
Before this commit: robot biped_s53, 32 links, 31 joints
Links:
- link waist_yaw_link: mass 23.55835568 -> 22.55935568
