Commit message: sync https://www.lejuhub.com/highlydynamic/kuavo-ros-control/commit/cceb80bcae7126e985c2dfea700ccf5e1b62466d

File: src/kuavo_assets/models/biped_s14/urdf/drake/biped_v3.urdf (robot description, URDF)
Before this commit: robot biped_v3, 14 links, 13 joints
Links:
- link torso: mass 12.097476 -> 13.500276

File: src/kuavo_assets/models/biped_s14/urdf/drake/biped_v3_all_joint.urdf (robot description, URDF)
Before this commit: robot biped_v3_all_joint, 30 links, 25 joints
Links:
- link torso: mass 6.89461242 -> 8.29741242

File: src/kuavo_assets/models/biped_s14/urdf/drake/biped_v3_full.urdf (robot description, URDF)
Before this commit: robot biped_v3_full, 22 links, 21 joints
Links:
- link torso: mass 9.385076 -> 10.787876

File: src/kuavo_assets/models/biped_s17/urdf/drake/biped_v3.urdf (robot description, URDF)
Before this commit: robot biped_v3, 14 links, 13 joints
Links:
- link torso: mass 15.78214703 -> 16.56814703

File: src/kuavo_assets/models/biped_s17/urdf/drake/biped_v3_all_joint.urdf (robot description, URDF)
Before this commit: robot biped_v3_all_joint, 30 links, 25 joints
Links:
- link torso: mass 8.98734703 -> 9.77334703

File: src/kuavo_assets/models/biped_s17/urdf/drake/biped_v3_full.urdf (robot description, URDF)
Before this commit: robot biped_v3_full, 22 links, 21 joints
Links:
- link torso: mass 9.63014703 -> 10.41614703
