Commit message: sync https://www.lejuhub.com/highlydynamic/kuavo-ros-control/commit/93657ebb00c795b1f9d96f2edb0e105703466d37

File: src/kuavo_assets/models/biped_s52/urdf/biped_s52.urdf (robot description, URDF)
Before this commit: robot biped_s52, 51 links, 50 joints
Links:
- removed link camera_base
Joints:
- removed joint camera_base_joint

File: src/kuavo_assets/models/biped_s52/urdf/biped_s52_gazebo.urdf (robot description, URDF)
Before this commit: robot biped_s52, 51 links, 50 joints
Links:
- removed link camera_base
- link head_camera_base: geometry visual mesh filename=package://kuavo_assets/models/biped_s52/meshes/head_camera_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
- link head_camera_depth: geometry visual mesh filename=package://kuavo_assets/models/biped_s52/meshes/head_camera_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
- link head_radar: geometry visual mesh filename=package://kuavo_assets/models/biped_s52/meshes/head_radar.S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
Joints:
- removed joint camera_base_joint

File: src/kuavo_assets/models/biped_s53/urdf/biped_s53.urdf (robot description, URDF)
Before this commit: robot biped_s53, 51 links, 50 joints
Links:
- removed link camera_base
Joints:
- removed joint camera_base_joint

File: src/kuavo_assets/models/biped_s53/urdf/biped_s53_gazebo.urdf (robot description, URDF)
Before this commit: robot biped_s53, 51 links, 50 joints
Links:
- removed link camera_base
- link base_link: geometry visual mesh filename=package://kuavo_assets/models/biped_s53/meshes/torso.STL
- link head_camera_base: geometry visual mesh filename=package://kuavo_assets/models/biped_s53/meshes/head_camera_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
- link head_camera_depth: geometry visual mesh filename=package://kuavo_assets/models/biped_s53/meshes/head_camera_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
- link head_radar: geometry visual mesh filename=package://kuavo_assets/models/biped_s53/meshes/head_radar.S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
- link leg_l1_link: geometry visual mesh filename=package://kuavo_assets/models/biped_s53/meshes/l_leg_roll.S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
- link leg_l2_link: geometry visual mesh filename=package://kuavo_assets/models/biped_s53/meshes/l_leg_yaw.STL
- link leg_l3_link: geometry visual mesh filename=package://kuavo_assets/models/biped_s53/meshes/l_leg_pitch.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
- link leg_l4_link: geometry visual mesh filename=package://kuavo_assets/models/biped_s53/meshes/l_knee.STL
- link leg_l5_link: geometry visual mesh filename=package://kuavo_assets/models/biped_s53/meshes/l_foot_pitch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
- link leg_l6_link: geometry collision box size=0.25 0.1 0.04; visual mesh filename=package://kuavo_assets/models/biped_s53/meshes/l_foot_roll.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
- link leg_r1_link: geometry visual mesh filename=package://kuavo_assets/models/biped_s53/meshes/r_leg_roll.S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
- link leg_r2_link: geometry visual mesh filename=package://kuavo_assets/models/biped_s53/meshes/r_leg_yaw.STL
- link leg_r3_link: geometry visual mesh filename=package://kuavo_assets/models/biped_s53/meshes/r_leg_pitch.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
- link leg_r4_link: geometry visual mesh filename=package://kuavo_assets/models/biped_s53/meshes/r_knee.STL
- link leg_r5_link: geometry visual mesh filename=package://kuavo_assets/models/biped_s53/meshes/r_foot_pitch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
- link leg_r6_link: geometry collision box size=0.25 0.1 0.04; visual mesh filename=package://kuavo_assets/models/biped_s53/meshes/r_foot_roll.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
- link waist_camera: geometry visual mesh filename=package://kuavo_assets/models/biped_s53/meshes/waist_camera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
- link waist_camera_base: geometry visual mesh filename=package://kuavo_assets/models/biped_s53/meshes/waist_camera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
- link waist_yaw_link: geometry visual mesh filename=package://kuavo_assets/models/biped_s53/meshes/waist_yaw.STL
- link zarm_l1_link: geometry visual mesh filename=package://kuavo_assets/models/biped_s53/meshes/l_arm_pitch.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
- link zarm_l2_link: geometry visual mesh filename=package://kuavo_assets/models/biped_s53/meshes/l_arm_roll.S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
- link zarm_l3_link: geometry visual mesh filename=package://kuavo_assets/models/biped_s53/meshes/l_arm_yaw.STL
- link zarm_l4_link: geometry visual mesh filename=package://kuavo_assets/models/biped_s53/meshes/l_forearm.STL
- link zarm_l5_link: geometry visual mesh filename=package://kuavo_assets/models/biped_s53/meshes/l_hand_yaw.S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
- link zarm_l6_link: geometry visual mesh filename=package://kuavo_assets/models/biped_s53/meshes/l_hand_roll.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
- link zarm_l7_link: geometry visual mesh filename=package://kuavo_assets/models/biped_s53/meshes/l_hand_pitch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
- link zarm_r1_link: geometry visual mesh filename=package://kuavo_assets/models/biped_s53/meshes/r_arm_pitch.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
- link zarm_r2_link: geometry visual mesh filename=package://kuavo_assets/models/biped_s53/meshes/r_arm_roll.S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
- link zarm_r3_link: geometry visual mesh filename=package://kuavo_assets/models/biped_s53/meshes/r_arm_yaw.STL
- link zarm_r4_link: geometry visual mesh filename=package://kuavo_assets/models/biped_s53/meshes/r_forearm.STL
- link zarm_r5_link: geometry visual mesh filename=package://kuavo_assets/models/biped_s53/meshes/r_hand_yaw.S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
- link zarm_r6_link: geometry visual mesh filename=package://kuavo_assets/models/biped_s53/meshes/r_hand_roll.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
- link zarm_r7_link: geometry collision box size=0.08 0.05 0.16; collision cylinder length=0.08 radius=0.01
- link zhead_1_link: geometry visual mesh filename=package://kuavo_assets/models/biped_s53/meshes/head_yaw.STL
- link zhead_2_link: geometry visual mesh filename=package://kuavo_assets/models/biped_s53/meshes/head_pitch.S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
Joints:
- removed joint camera_base_joint

File: src/kuavo_assets/models/biped_s54/urdf/biped_s54.urdf (robot description, URDF)
Before this commit: robot biped_s54, 51 links, 50 joints
Links:
- removed link camera_base
Joints:
- removed joint camera_base_joint

File: src/kuavo_assets/models/biped_s54/urdf/biped_s54_gazebo.urdf (robot description, URDF)
Before this commit: robot biped_s54, 51 links, 50 joints
Links:
- removed link camera_base
- link base_link: geometry visual mesh filename=package://kuavo_assets/models/biped_s54/meshes/torso.STL
- link head_camera_base: geometry visual mesh filename=package://kuavo_assets/models/biped_s54/meshes/head_camera_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
- link head_camera_depth: geometry visual mesh filename=package://kuavo_assets/models/biped_s54/meshes/head_camera_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
- link head_radar: geometry visual mesh filename=package://kuavo_assets/models/biped_s54/meshes/head_radar.S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
- link leg_l1_link: geometry visual mesh filename=package://kuavo_assets/models/biped_s54/meshes/l_leg_roll.S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
- link leg_l2_link: geometry visual mesh filename=package://kuavo_assets/models/biped_s54/meshes/l_leg_yaw.STL
- link leg_l3_link: geometry visual mesh filename=package://kuavo_assets/models/biped_s54/meshes/l_leg_pitch.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
- link leg_l4_link: geometry visual mesh filename=package://kuavo_assets/models/biped_s54/meshes/l_knee.STL
- link leg_l5_link: geometry visual mesh filename=package://kuavo_assets/models/biped_s54/meshes/l_foot_pitch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
- link leg_l6_link: geometry collision box size=0.25 0.1 0.04; visual mesh filename=package://kuavo_assets/models/biped_s54/meshes/l_foot_roll.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
- link leg_r1_link: geometry visual mesh filename=package://kuavo_assets/models/biped_s54/meshes/r_leg_roll.S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
- link leg_r2_link: geometry visual mesh filename=package://kuavo_assets/models/biped_s54/meshes/r_leg_yaw.STL
- link leg_r3_link: geometry visual mesh filename=package://kuavo_assets/models/biped_s54/meshes/r_leg_pitch.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
- link leg_r4_link: geometry visual mesh filename=package://kuavo_assets/models/biped_s54/meshes/r_knee.STL
- link leg_r5_link: geometry visual mesh filename=package://kuavo_assets/models/biped_s54/meshes/r_foot_pitch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
- link leg_r6_link: geometry collision box size=0.25 0.1 0.04; visual mesh filename=package://kuavo_assets/models/biped_s54/meshes/r_foot_roll.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
- link waist_camera: geometry visual mesh filename=package://kuavo_assets/models/biped_s54/meshes/waist_camera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
- link waist_camera_base: geometry visual mesh filename=package://kuavo_assets/models/biped_s54/meshes/waist_camera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
- link waist_yaw_link: geometry visual mesh filename=package://kuavo_assets/models/biped_s54/meshes/waist_yaw.STL
- link zarm_l1_link: geometry visual mesh filename=package://kuavo_assets/models/biped_s54/meshes/l_arm_pitch.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
- link zarm_l2_link: geometry visual mesh filename=package://kuavo_assets/models/biped_s54/meshes/l_arm_roll.S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
- link zarm_l3_link: geometry visual mesh filename=package://kuavo_assets/models/biped_s54/meshes/l_arm_yaw.STL
- link zarm_l4_link: geometry visual mesh filename=package://kuavo_assets/models/biped_s54/meshes/l_forearm.STL
- link zarm_l5_link: geometry visual mesh filename=package://kuavo_assets/models/biped_s54/meshes/l_hand_yaw.S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
- link zarm_l6_link: geometry visual mesh filename=package://kuavo_assets/models/biped_s54/meshes/l_hand_roll.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
- link zarm_l7_link: geometry visual mesh filename=package://kuavo_assets/models/biped_s54/meshes/l_hand_pitch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
- link zarm_r1_link: geometry visual mesh filename=package://kuavo_assets/models/biped_s54/meshes/r_arm_pitch.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
- link zarm_r2_link: geometry visual mesh filename=package://kuavo_assets/models/biped_s54/meshes/r_arm_roll.S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
- link zarm_r3_link: geometry visual mesh filename=package://kuavo_assets/models/biped_s54/meshes/r_arm_yaw.STL
- link zarm_r4_link: geometry visual mesh filename=package://kuavo_assets/models/biped_s54/meshes/r_forearm.STL
- link zarm_r5_link: geometry visual mesh filename=package://kuavo_assets/models/biped_s54/meshes/r_hand_yaw.S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
- link zarm_r6_link: geometry visual mesh filename=package://kuavo_assets/models/biped_s54/meshes/r_hand_roll.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
- link zarm_r7_link: geometry collision box size=0.08 0.05 0.16; collision cylinder length=0.08 radius=0.01
- link zhead_1_link: geometry visual mesh filename=package://kuavo_assets/models/biped_s54/meshes/head_yaw.STL
- link zhead_2_link: geometry visual mesh filename=package://kuavo_assets/models/biped_s54/meshes/head_pitch.S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
Joints:
- removed joint camera_base_joint

File: src/kuavo_assets/models/biped_s55/urdf/biped_s55.urdf (robot description, URDF)
Before this commit: robot biped_s55, 51 links, 50 joints
Links:
- removed link camera_base
Joints:
- removed joint camera_base_joint

File: src/kuavo_assets/models/biped_s55/urdf/biped_s55_gazebo.urdf (robot description, URDF)
Before this commit: robot biped_s55, 51 links, 50 joints
Links:
- removed link camera_base
- link base_link: geometry visual mesh filename=package://kuavo_assets/models/biped_s55/meshes/torso.STL
- link head_camera_base: geometry visual mesh filename=package://kuavo_assets/models/biped_s55/meshes/head_camera_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
- link head_camera_depth: geometry visual mesh filename=package://kuavo_assets/models/biped_s55/meshes/head_camera_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
- link head_radar: geometry visual mesh filename=package://kuavo_assets/models/biped_s55/meshes/head_radar.S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
- link leg_l1_link: geometry visual mesh filename=package://kuavo_assets/models/biped_s55/meshes/l_leg_roll.S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
- link leg_l2_link: geometry visual mesh filename=package://kuavo_assets/models/biped_s55/meshes/l_leg_yaw.STL
- link leg_l3_link: geometry visual mesh filename=package://kuavo_assets/models/biped_s55/meshes/l_leg_pitch.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
- link leg_l4_link: geometry visual mesh filename=package://kuavo_assets/models/biped_s55/meshes/l_knee.STL
- link leg_l5_link: geometry visual mesh filename=package://kuavo_assets/models/biped_s55/meshes/l_foot_pitch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
- link leg_l6_link: geometry collision box size=0.25 0.1 0.04; visual mesh filename=package://kuavo_assets/models/biped_s55/meshes/l_foot_roll.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
- link leg_r1_link: geometry visual mesh filename=package://kuavo_assets/models/biped_s55/meshes/r_leg_roll.S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
- link leg_r2_link: geometry visual mesh filename=package://kuavo_assets/models/biped_s55/meshes/r_leg_yaw.STL
- link leg_r3_link: geometry visual mesh filename=package://kuavo_assets/models/biped_s55/meshes/r_leg_pitch.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
- link leg_r4_link: geometry visual mesh filename=package://kuavo_assets/models/biped_s55/meshes/r_knee.STL
- link leg_r5_link: geometry visual mesh filename=package://kuavo_assets/models/biped_s55/meshes/r_foot_pitch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
- link leg_r6_link: geometry collision box size=0.25 0.1 0.04; visual mesh filename=package://kuavo_assets/models/biped_s55/meshes/r_foot_roll.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
- link waist_camera: geometry visual mesh filename=package://kuavo_assets/models/biped_s55/meshes/waist_camera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
- link waist_camera_base: geometry visual mesh filename=package://kuavo_assets/models/biped_s55/meshes/waist_camera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
- link waist_yaw_link: geometry visual mesh filename=package://kuavo_assets/models/biped_s55/meshes/waist_yaw.STL
- link zarm_l1_link: geometry visual mesh filename=package://kuavo_assets/models/biped_s55/meshes/l_arm_pitch.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
- link zarm_l2_link: geometry visual mesh filename=package://kuavo_assets/models/biped_s55/meshes/l_arm_roll.S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
- link zarm_l3_link: geometry visual mesh filename=package://kuavo_assets/models/biped_s55/meshes/l_arm_yaw.STL
- link zarm_l4_link: geometry visual mesh filename=package://kuavo_assets/models/biped_s55/meshes/l_forearm.STL
- link zarm_l5_link: geometry visual mesh filename=package://kuavo_assets/models/biped_s55/meshes/l_hand_yaw.S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
- link zarm_l6_link: geometry visual mesh filename=package://kuavo_assets/models/biped_s55/meshes/l_hand_roll.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
- link zarm_l7_link: geometry visual mesh filename=package://kuavo_assets/models/biped_s55/meshes/l_hand_pitch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
- link zarm_r1_link: geometry visual mesh filename=package://kuavo_assets/models/biped_s55/meshes/r_arm_pitch.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
- link zarm_r2_link: geometry visual mesh filename=package://kuavo_assets/models/biped_s55/meshes/r_arm_roll.S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
- link zarm_r3_link: geometry visual mesh filename=package://kuavo_assets/models/biped_s55/meshes/r_arm_yaw.STL
- link zarm_r4_link: geometry visual mesh filename=package://kuavo_assets/models/biped_s55/meshes/r_forearm.STL
- link zarm_r5_link: geometry visual mesh filename=package://kuavo_assets/models/biped_s55/meshes/r_hand_yaw.S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
- link zarm_r6_link: geometry visual mesh filename=package://kuavo_assets/models/biped_s55/meshes/r_hand_roll.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
- link zarm_r7_link: geometry collision box size=0.08 0.05 0.16; collision cylinder length=0.08 radius=0.01
- link zhead_1_link: geometry visual mesh filename=package://kuavo_assets/models/biped_s55/meshes/head_yaw.STL
- link zhead_2_link: geometry visual mesh filename=package://kuavo_assets/models/biped_s55/meshes/head_pitch.S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
Joints:
- removed joint camera_base_joint

File: src/kuavo_assets/models/biped_s55/urdf/biped_s55_gazebo.xacro (robot description, xacro)
@@ -6,5 +6,5 @@
   <xacro:include filename="$(find realsense_ros_gazebo)/xacro/depthcam.xacro"/>
   <!-- d435 声明 -->
-  <xacro:realsense_d435 sensor_name="camera" parent_link="camera_base" rate="30">
+  <xacro:realsense_d435 sensor_name="camera" parent_link="head_camera_base" rate="30">
     <origin rpy="0 0 0 " xyz="0 0 0"/>
   </xacro:realsense_d435>

File: src/kuavo_assets/models/biped_s61/urdf/biped_s61.urdf (robot description, URDF)
Before this commit: robot biped_s61, 36 links, 35 joints
Links:
- removed link camera
- removed link camera_base
- added link head_camera_base, mass 0.0482361371130408; visual mesh filename=package://kuavo_assets/models/biped_s61/meshes/head_camera.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
- added link head_camera_depth, mass 0.0482361371130408
Joints:
- removed joint camera
- removed joint camera_base_joint
- added joint head_camera_base_joint: type fixed, parent zhead_2_link, child head_camera_base, origin xyz=0.099619 0 0.032844 rpy=0 0.3406 0
- added joint head_camera_depth_joint: type fixed, parent head_camera_base, child head_camera_depth, origin xyz=0.011715 0.0475 0.014311 rpy=0 0 0

File: src/kuavo_assets/models/biped_s61/urdf/biped_s61_gazebo.urdf (robot description, URDF)
Before this commit: robot biped_s61, 39 links, 38 joints
Links:
- removed link camera
- added link head_camera_base, mass 0.001; visual mesh filename=package://kuavo_assets/models/biped_s61/meshes/head_camera.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
- added link head_camera_depth, mass 0.001
Joints:
- removed joint camera
- added joint head_camera_base_joint: type fixed, parent zhead_2_link, child head_camera_base, origin xyz=0.099619 0 0.032844 rpy=0 0.3406 0
- added joint head_camera_depth_joint: type fixed, parent head_camera_base, child head_camera_depth, origin xyz=0.011715 0.0475 0.014311 rpy=0 0 0

File: src/kuavo_assets/models/biped_s62/urdf/biped_s62.urdf (robot description, URDF)
Before this commit: robot biped_s62, 36 links, 35 joints
Links:
- removed link camera
- removed link camera_base
- added link head_camera_base, mass 0.0482361371130408; visual mesh filename=package://kuavo_assets/models/biped_s62/meshes/head_camera.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
- added link head_camera_depth, mass 0.0482361371130408
Joints:
- removed joint camera
- removed joint camera_base_joint
- added joint head_camera_base_joint: type fixed, parent zhead_2_link, child head_camera_base, origin xyz=0.099619 0 0.032844 rpy=0 0.3406 0
- added joint head_camera_depth_joint: type fixed, parent head_camera_base, child head_camera_depth, origin xyz=0.011715 0.0475 0.014311 rpy=0 0 0

File: src/kuavo_assets/models/biped_s62/urdf/biped_s62_gazebo.urdf (robot description, URDF)
Before this commit: robot biped_s62, 39 links, 38 joints
Links:
- removed link camera
- added link head_camera_base, mass 0.001; visual mesh filename=package://kuavo_assets/models/biped_s62/meshes/head_camera.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
- added link head_camera_depth, mass 0.001
Joints:
- removed joint camera
- added joint head_camera_base_joint: type fixed, parent zhead_2_link, child head_camera_base, origin xyz=0.099619 0 0.032844 rpy=0 0.3406 0
- added joint head_camera_depth_joint: type fixed, parent head_camera_base, child head_camera_depth, origin xyz=0.011715 0.0475 0.014311 rpy=0 0 0

File: src/kuavo_assets/models/biped_s62/urdf/biped_s62_gazebo.xacro (robot description, xacro)
@@ -5,5 +5,5 @@
   <!-- 可选：深度相机（如不需要可移除本段） -->
   <xacro:include filename="$(find realsense_ros_gazebo)/xacro/depthcam.xacro"/>
-  <xacro:realsense_d435 sensor_name="camera" parent_link="camera" rate="30">
+  <xacro:realsense_d435 sensor_name="camera" parent_link="head_camera_base" rate="30">
     <origin rpy="0 0 0" xyz="0 0 0"/>
   </xacro:realsense_d435>

File: src/kuavo_assets/models/biped_s63/urdf/biped_s63.urdf (robot description, URDF)
Before this commit: robot biped_s63, 36 links, 35 joints
Links:
- removed link camera
- removed link camera_base
- added link head_camera_base, mass 0.0; visual mesh filename=package://kuavo_assets/models/biped_s63/meshes/head_camera_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
- added link head_camera_depth, mass 0.0; visual mesh filename=package://kuavo_assets/models/biped_s63/meshes/head_camera_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
Joints:
- removed joint camera
- removed joint camera_base_joint
- added joint head_camera_base_joint: type fixed, parent zhead_2_link, child head_camera_base, origin xyz=0.099619 0 0.032844 rpy=0 0.3406 0
- added joint head_camera_depth_joint: type fixed, parent head_camera_base, child head_camera_depth, origin xyz=0.011715 0.0475 0.014311 rpy=0 0 0

File: src/kuavo_assets/models/biped_s63/urdf/biped_s63_gazebo.urdf (robot description, URDF)
Before this commit: robot biped_s63, 39 links, 38 joints
Links:
- removed link camera
- added link head_camera_base, mass 0.0; visual mesh filename=package://kuavo_assets/models/biped_s63/meshes/head_camera_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
- added link head_camera_depth, mass 0.0; visual mesh filename=package://kuavo_assets/models/biped_s63/meshes/head_camera_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
- link waist_yaw_link: geometry visual mesh filename=package://kuavo_assets/models/biped_s63/meshes/torso.STL
Joints:
- removed joint camera
- added joint head_camera_base_joint: type fixed, parent zhead_2_link, child head_camera_base, origin xyz=0.099619 0 0.032844 rpy=0 0.3406 0
- added joint head_camera_depth_joint: type fixed, parent head_camera_base, child head_camera_depth, origin xyz=0.011715 0.0475 0.014311 rpy=0 0 0

File: src/kuavo_assets/models/biped_s63/urdf/biped_s63_gazebo.xacro (robot description, xacro)
@@ -5,5 +5,5 @@
   <!-- 可选：深度相机（如不需要可移除本段） -->
   <xacro:include filename="$(find realsense_ros_gazebo)/xacro/depthcam.xacro"/>
-  <xacro:realsense_d435 sensor_name="camera" parent_link="camera" rate="30">
+  <xacro:realsense_d435 sensor_name="camera" parent_link="head_camera_base" rate="30">
     <origin rpy="0 0 0" xyz="0 0 0"/>
   </xacro:realsense_d435>
